Commit message: Added Sonars

File: robots/mp_500/mp_500.urdf.xacro (robot description, xacro)
@@ -6,122 +6,91 @@
   <!-- MATERIALS -->
   <xacro:include filename="$(find neo_simulation)/robots/mp_500/xacros/mp_500_materials.xacro" />
-<!--++++++++++++++++++++++++++++++base_link++++++++++++++++++++++++++++++++++++++++++++++++++++-->
-<!--++++++++++++++++++++body++++++++++++++++++++++++++++-->
+	<!--++++++++++++++++++++++++++++++base_link++++++++++++++++++++++++++++++++++++++++++++++++++++-->
+	<!--++++++++++++++++++++body++++++++++++++++++++++++++++-->
 	<link name="base_link">
-      <!--inertial>
-        <mass value="67.010" />
-        <origin xyz="0.0 0.0 0.234" rpy="0 0 0"/>
-        <inertia ixx="1417853.715" ixy="17813.155" ixz="-21078.206"
-                 iyy="2030191.708" iyz="-4813.295"
-                 izz="2180211.662" />
-      </inertial-->
-	  <inertial>
-		  <mass value="5.67" />
-		    <origin xyz="0 0 0.0" rpy="0 0 0"/>
-		    <inertia ixx="0.07" ixy="0.0" ixz="0.0"
-		             iyy="0.08" iyz="0.0"
-		             izz="0.1" />
-	  </inertial>
-      <visual name='body'>
-        <!--origin xyz="0.0 0.0 0.234" rpy="0 0 1.57" /--><!-- for cylinder -->
-		<origin xyz="0.0 0.0 0.08" rpy="0 0 1.57" /><!-- for STL -->
-        <geometry>
-            <mesh filename="package://neo_simulation/robots/mp_500/meshes/base.stl" scale="1 1 1"/>
-	    	<!--cylinder length="0.381" radius="0.2545"/-->
-	    	<!--box size="0.445 0.277 0.17"/-->
-        </geometry>
-        <material name="Neobotix/Grey" />
-      </visual>
-      <collision name='body_collision'>
-        <origin xyz="0.0 0.0 0.234" rpy="0 0 0" />
-        <geometry>
-          <box size="0.4 0.600 0.400"/> <!--TODO: Find correct values-->
-          <!--cylinder length="0.381" radius="0.2545"/-->
-        </geometry>
-      </collision>
-<!--+++++++++++++++++++castor_front++++++++++++++++++++++++-->
-	<!--<visual name='castor_front_visual'>
-          <origin xyz="0.2 0 0.018" rpy="0 0 0" />
-          <geometry>
-            <sphere radius="0.016"/>
-          </geometry>
-          <material name="Neobotix/Black" />
-      </visual>
-      <collision name='castor_front_collision'>
-	  	<origin xyz="0.2 0 0.018 " rpy="0 0 0" />
-          <geometry>
-            <sphere radius="0.016"/>
-          </geometry>
-    </collision>-->
-<!--+++++++++++++++++++castor_back++++++++++++++++++++++++-->
-	<visual name='castor_back_visual'>
-          <origin xyz="-0.47 0 0.0161" rpy="0 0 0" />
-          <geometry>
-            <sphere radius="0.016"/>
-          </geometry>
-          <material name="Neobotix/Black" />
-      </visual>
-      <collision name='castor_back_collision'>
-	  	<origin xyz="-0.47 0 0.0161 " rpy="0 0 0" />
-          <geometry>
-            <sphere radius="0.016"/>
-          </geometry>
-       </collision>
-    </link>
-<!--+++++++++++++++++++wheel_left_link++++++++++++++++++++++++-->
-<link name="wheel_left_link" type="wheel">
-    <inertial>
-      <mass value="1.5" />
-      <origin xyz="0.0 0.0 -0.0" rpy="0 0 0" />
-      <inertia ixx="0.0051" ixy="0" ixz="0" iyy="0.0051" iyz="0" izz="0.009" />
-    </inertial>
-    <visual>
-     	<origin xyz="0.0 0.0 -0.00" rpy="0 0 0" />
-     	<geometry>
-			<cylinder radius="0.13" length="0.08"/>
-     	</geometry>
-     	<material name="Neobotix/Black" />
-    </visual>
-     <!-- <visual>
-	<origin xyz="0.0 0.0 0.08" rpy="0 0 0" />
-        <geometry>
-            <mesh filename="package://neo_simulation/robots/mp_500/meshes/wheel.stl"/>
-        </geometry>
-        <material name="Neobotix/Grey" />
-      </visual>-->
-    <collision>
-     	<origin xyz="0.0 0.0 0.0" rpy="0 0 0" />
-     	<geometry>
-        	<cylinder radius="0.13" length="0.08"/>
-     	</geometry>
-    </collision>
-</link>
-<!--+++++++++++++++++++wheel_left_joint++++++++++++++++++++++++-->
-	<joint name="wheel_left_joint" type="revolute">
-		<origin xyz="0 -0.2645 0.13" rpy="0 1.57 1.57" />
-    	<axis xyz="0 0 1"/>
-    	<limit effort="1000.0" lower="-1e+16" upper="1e+16" velocity="3.5"/>
-    	<joint_properties damping="0.0" friction="0.0" />
-    	<parent link="base_link" />
-    	<child link="wheel_left_link" />
-    </joint>
+		<inertial>
+			<mass value="5.67" />
+			<origin xyz="0 0 0.0" rpy="0 0 0"/>
+			<inertia ixx="0.07" ixy="0.0" ixz="0.0"
+				     iyy="0.08" iyz="0.0"
+				     izz="0.1" />
+		</inertial>
+	      <visual name='body'>
+			<origin xyz="0.0 0.0 0.075" rpy="0 0 1.57" /><!-- for STL -->
+		<geometry>
+		    <mesh filename="package://neo_simulation/robots/mp_500/meshes/base.stl" scale="1 1 1"/>
+		</geometry>
+		<material name="Neobotix/Grey" />
+	      </visual>
+	      <collision name='body_collision'>
+		<origin xyz="-0.183 0.0 0.234" rpy="0 0 0" />
+		<geometry>
+		  <box size="0.734 0.600 0.400"/>
+		  <!--cylinder length="0.381" radius="0.2545"/-->
+		</geometry>
+	      </collision>
+		  <!--    <visual name='box_visual'>
+		  <origin xyz="-0.183 0.0 0.234" rpy="0 0 0" />
+		  <geometry>
+		    <box size="0.734 0.600 0.400"/>
+		  </geometry>
+		  <material name="Neobotix/Black" />
+	      </visual>-->
+	<!--+++++++++++++++++++castor_back++++++++++++++++++++++++-->
+	      <collision name='castor_back_collision'>
+		  	<origin xyz="-0.47 0 0.0161 " rpy="0 0 0" />
+		  <geometry>
+		    <sphere radius="0.016"/>
+		  </geometry>
+	       </collision>
+	</link>
+	<!--+++++++++++++++++++wheel_left_link++++++++++++++++++++++++-->
+	<link name="wheel_left_link" type="wheel">
+	    <inertial>
+	      <mass value="1.5" />
+	      <origin xyz="0.0 0.0 -0.0" rpy="0 0 0" />
+	      <inertia ixx="0.0051" ixy="0" ixz="0" iyy="0.0051" iyz="0" izz="0.009" />
+	    </inertial>
+	    <!--<visual>
+	     	<origin xyz="0.0 0.0 -0.00" rpy="0 0 0" />
+	     	<geometry>
+				<cylinder radius="0.13" length="0.085"/>
+	     	</geometry>
+	     	<material name="Neobotix/Black" />
+	    </visual>-->
+	    <collision>
+	     	<origin xyz="0.0 0.0 0.0" rpy="0 0 0" />
+	     	<geometry>
+			<cylinder radius="0.13" length="0.085"/>
+	     	</geometry>
+	    </collision>
+	</link>
+	<!--+++++++++++++++++++wheel_left_joint++++++++++++++++++++++++-->
+		<joint name="wheel_left_joint" type="revolute">
+			<origin xyz="0 -0.2534 0.119" rpy="0 1.57 1.57" />
+	    	<axis xyz="0 0 1"/>
+	    	<limit effort="1000.0" lower="-1e+16" upper="1e+16" velocity="3.5"/>
+	    	<joint_properties damping="0.0" friction="0.0" />
+	    	<parent link="base_link" />
+	    	<child link="wheel_left_link" />
+	    </joint>
 	<!--+++++++++++++++++++wheel_right_link++++++++++++++++++++++++-->
 	<link name="wheel_right_link" type="wheel">
 		<inertial>
-		  <mass value="1.5" />
+	      	  <mass value="1.5" />
 		  <origin xyz="0 0.0 0.0" rpy="0 0 0" />
 		  <inertia ixx="0.0051" ixy="0" ixz="0" iyy="0.0051" iyz="0" izz="0.009" />
 		</inertial>
-		<visual>
-		 	<origin xyz="0 0.0 0.016" rpy="0 0 0" />
+		<!--<visual>
+		 	<origin xyz="0 0.0 0.0" rpy="0 0 0" />
 		 	<geometry>
-				<cylinder radius="0.13" length="0.08"/>
+			<cylinder radius="0.13" length="0.085"/>
 		 	</geometry>
 		 	<material name="Neobotix/Black" />
-		</visual>
+		</visual>-->
 		<collision>
-		 	<origin xyz="0.0 0.0 0.00" rpy="0 0 0" />
+			<origin xyz="0.0 0.0 0.00" rpy="0 0 0" />
 		 	<geometry>
-		    	<cylinder radius="0.13" length="0.08"/>
+			    	<cylinder radius="0.13" length="0.085"/>
 		 	</geometry>
 		</collision>
@@ -129,20 +98,20 @@
 	<!--+++++++++++++++++++wheel_right_joint++++++++++++++++++++++++-->
 	<joint name="wheel_right_joint" type="revolute">
-    	<origin xyz="0 0.2645 0.13" rpy="0 1.57 1.57" />
-    	<axis xyz="0 0 1"/>
-    	<limit effort="1000.0" lower="-1e+16" upper="1e+16" velocity="3.5"/>
-    	<joint_properties damping="0.0" friction="0.0" />
-    	<parent link="base_link" />
-    	<child link="wheel_right_link" />
-    </joint>
+	   <origin xyz="0 0.2534 0.119" rpy="0 1.57 1.57" />
+	   <axis xyz="0 0 1"/>
+	   <limit effort="1000.0" lower="-1e+16" upper="1e+16" velocity="3.5"/>
+	   <joint_properties damping="0.0" friction="0.0" />
+	   <parent link="base_link" />
+	   <child link="wheel_right_link" />
+	</joint>
 	<!--+++++++++++++++++++laserscanner_front_joint++++++++++++++++++++++++-->
-	<joint name="laserscanner_front_joint" type="fixed">
-		  <axis xyz="0 1 0" />
-		  <origin xyz="0.244 0 0.141" rpy="3.14 0 0" />
-		  <parent link="base_link"/>
-		  <child link="laserscanner_front_link"/>
+	<joint name="scanner_front_joint" type="fixed">
+	  <axis xyz="0 1 0" />
+	  <origin xyz="0.244 0 0.141" rpy="3.14 0 0" />
+	  <parent link="base_link"/>
+	  <child link="scanner_front_link"/>
 	</joint>
 	<!--+++++++++++++++++++laserscanner_front_link++++++++++++++++++++++++-->
-	<link name="laserscanner_front_link" type="laser">
+	<link name="scanner_front_link" type="laser">
 		<inertial>
 			<mass value="0.001" />
@@ -150,17 +119,57 @@
 			<inertia ixx="0.0001" ixy="0" ixz="0" iyy="0.000001" iyz="0" izz="0.0001" />
 	  	</inertial>
-	  	<visual>
+	<!--  	<visual>
 			<origin xyz="0 0 -0.04" rpy="0 0 -1.57" />
 			<geometry>
-		  		<mesh filename="package://neo_mp_500/robot_model/mp_500/meshes/SICK-S300.STL" />
+		  		<mesh filename="package://neo_simulation/robots/mp_500/meshes/SICK-S300.STL" />
 			</geometry>
 			<material name="Neobotix/Yellow" />
-	  	</visual>
+	  	</visual>-->
 	  	<collision>
 			<origin xyz="0 0 0" rpy="0 0 0" />
 			<geometry>
-		  	<cylinder length="0.154" radius="0.053" />
+				<cylinder length="0.154" radius="0.053" />
 			</geometry>
-	  	</collision>
+		  </collision>
 	</link>
+	<!--+++++++++++++++++++sonar_fr_joint++++++++++++++++++++++++-->
+	<joint name="sonar_fr_joint" type="fixed">
+	  <origin xyz="0.20116 -0.140 0.29948" rpy="0 -${pi/6} 0" />
+	  <parent link="base_link"/>
+	  <child link="sonar_fr_link"/>
+	</joint>
+	<!--+++++++++++++++++++sonar_fr_link++++++++++++++++++++++++-->
+	<link name="sonar_fr_link" type="sonar"/>
+	<!--+++++++++++++++++++sonar_fl_joint++++++++++++++++++++++++-->
+	<joint name="sonar_fl_joint" type="fixed">
+	  <origin xyz="0.20116 0.140 0.29948" rpy="0 -${pi/6} 0" />
+	  <parent link="base_link"/>
+	  <child link="sonar_fl_link"/>
+	</joint>
+	<!--+++++++++++++++++++sonar_fl_link++++++++++++++++++++++++-->
+	<link name="sonar_fl_link" type="sonar"/>
+	<!--+++++++++++++++++++sonar_bc_joint++++++++++++++++++++++++-->
+	<joint name="sonar_bc_joint" type="fixed">
+	  <origin xyz="-0.51116 0 0.29948" rpy="${pi} -${pi/6 + 2* pi/3} 0" />
+	  <parent link="base_link"/>
+	  <child link="sonar_bc_link"/>
+	</joint>
+	<!--+++++++++++++++++++sonar_bc_link++++++++++++++++++++++++-->
+	<link name="sonar_bc_link" type="sonar"/>
+	<!--+++++++++++++++++++sonar_br_joint++++++++++++++++++++++++-->
+	<joint name="sonar_br_joint" type="fixed">
+	  <origin xyz="-0.454192 0.122993 0.29948" rpy="0 -${pi/6} ${122/180 *pi}" />
+	  <parent link="base_link"/>
+	  <child link="sonar_br_link"/>
+	</joint>
+	<!--+++++++++++++++++++sonar_br_link++++++++++++++++++++++++-->
+	<link name="sonar_br_link" type="sonar"/>
+	<!--+++++++++++++++++++sonar_bl_joint++++++++++++++++++++++++-->
+	<joint name="sonar_bl_joint" type="fixed">
+	  <origin xyz="-0.454192 -0.122993 0.29948" rpy="0 -${pi/6} -${122/180 *pi}" />
+	  <parent link="base_link"/>
+	  <child link="sonar_bl_link"/>
+	</joint>
+	<!--+++++++++++++++++++sonar_bl_link++++++++++++++++++++++++-->
+	<link name="sonar_bl_link" type="sonar"/>
 </robot>

File: robots/mp_500/xacros/mp_500_gazebo.xacro (robot description, xacro)
@@ -73,5 +73,5 @@
       <leftJoint>wheel_left_joint</leftJoint>
       <rightJoint>wheel_right_joint</rightJoint>
-      <wheelSeparation>0.5390</wheelSeparation>
+      <wheelSeparation>0.5068</wheelSeparation>
       <wheelDiameter>0.26</wheelDiameter>
       <torque>1</torque>
